File: batteryboard-bottom/batteryboard-bottom.kicad_sch (KiCad schematic)
At the start: 6 parts

Commit message: labeled connections
Connections:
- net GND: now also J?.4 (Pin_4), J?.4 (Pin_4)
- net BATT_P_SW: now reaches J?.1 (Pin_1), J?.1 (Pin_1)
- net BURN2: now reaches J?.10 (Pin_10), J?.10 (Pin_10)
- net BATT_P: now reaches J?.11 (Pin_11), J?.11 (Pin_11)
- net VBUS: now reaches J?.12 (Pin_12), J?.12 (Pin_12)
- net BATT_N_SW: now reaches J?.2 (Pin_2), J?.2 (Pin_2)
- net +3V3: now reaches J?.3 (Pin_3), J?.3 (Pin_3)
- net SDA3: now reaches J?.5 (Pin_5), J?.5 (Pin_5)
- net SCL3: now reaches J?.6 (Pin_6), J?.6 (Pin_6)
- net COIL_P: now reaches J?.7 (Pin_7), J?.7 (Pin_7)
- net COIL_N: now reaches J?.8 (Pin_8), J?.8 (Pin_8)
- net BURN1: now reaches J?.9 (Pin_9), J?.9 (Pin_9)
Other:
- note added: "bottom batteryboard"
- note removed: "batteryboard"
Changed lines of the file:
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@@
     (effects (font (size 2.54 2.54)) (justify left bottom))
   )
-  (text "batteryboard" (at 124.714 114.681 0)
+  (text "bottom batteryboard" (at 111.76 114.3 0)
     (effects (font (size 3.9878 3.9878) (thickness 1.016) bold) (justify left bottom))
   )
@@
     (effects (font (size 2.54 2.54)) (justify left bottom))
   )
+  (label "+3V3" (at 83.82 43.18 0)
+    (effects (font (size 1.27 1.27)) (justify left bottom))
+  )
+  (label "SCL3" (at 83.82 50.8 0)
+    (effects (font (size 1.27 1.27)) (justify left bottom))
+  )
+  (label "COIL_P" (at 83.82 53.34 0)
+    (effects (font (size 1.27 1.27)) (justify left bottom))
+  )
+  (label "BATT_N_SW" (at 83.82 40.64 0)
+    (effects (font (size 1.27 1.27)) (justify left bottom))
+  )
+  (label "COIL_N" (at 83.82 55.88 0)
+    (effects (font (size 1.27 1.27)) (justify left bottom))
+  )
+  (label "GND" (at 83.82 45.72 0)
+    (effects (font (size 1.27 1.27)) (justify left bottom))
+  )
+  (label "VBUS" (at 83.82 66.04 0)
+    (effects (font (size 1.27 1.27)) (justify left bottom))
+  )
+  (label "BATT_P" (at 83.82 63.5 0)
+    (effects (font (size 1.27 1.27)) (justify left bottom))
+  )
+  (label "SDA3" (at 83.82 48.26 0)
+    (effects (font (size 1.27 1.27)) (justify left bottom))
+  )
+  (label "BATT_P_SW" (at 83.82 38.1 0)
+    (effects (font (size 1.27 1.27)) (justify left bottom))
+  )
+  (label "BURN2" (at 83.82 60.96 0)
+    (effects (font (size 1.27 1.27)) (justify left bottom))
+  )
+  (label "BURN1" (at 83.82 58.42 0)
+    (effects (font (size 1.27 1.27)) (justify left bottom))
+  )
   (symbol (lib_id "Connector_Generic:Conn_01x12") (at 144.78 50.8 0) (unit 1)

Commit message: switch to 2x connectors for battery boards
Parts:
- removed J?: Conn_01x12, symbol Connector_Generic:Conn_01x12
- added J?: Conn_02x06_Odd_Even, symbol Connector_Generic:Conn_02x06_Odd_Even
Connections:
- net +3V3: now also J?.3 (Pin_3)
- net BATT_N_SW: now also J?.2 (Pin_2)
- net BATT_P: now also J?.11 (Pin_11)
- net BATT_P_SW: now also J?.1 (Pin_1)
- net BURN1: now also J?.9 (Pin_9)
- net BURN2: now also J?.10 (Pin_10)
- net COIL_N: now also J?.8 (Pin_8)
- net COIL_P: now also J?.7 (Pin_7)
- net GND: now also J?.4 (Pin_4)
- net SCL3: now also J?.6 (Pin_6)
- net SDA3: now also J?.5 (Pin_5)
- net VBUS: now also J?.12 (Pin_12)
Other:
- note removed: "Grounded Mounting Holes"

Commit message: remove burn wire signals
Parts:
- removed J?: Conn_02x06_Odd_Even, symbol Connector_Generic:Conn_02x06_Odd_Even
- removed J?: Conn_01x12, symbol Connector_Generic:Conn_01x12
- added J?: Conn_02x05_Odd_Even, symbol Connector_Generic:Conn_02x05_Odd_Even
- added J?: Conn_01x10, symbol Connector_Generic:Conn_01x10
Connections:
- net +3V3: now also J?.3 (Pin_3), J?.3 (Pin_3)
- net BATT_N_SW: now also J?.2 (Pin_2), J?.2 (Pin_2)
- net BATT_P: now also J?.9 (Pin_9), J?.9 (Pin_9)
- net BATT_P_SW: now also J?.1 (Pin_1), J?.1 (Pin_1)
- net COIL_N: now also J?.8 (Pin_8), J?.8 (Pin_8)
- net COIL_P: now also J?.7 (Pin_7), J?.7 (Pin_7)
- net GND: now also J?.4 (Pin_4), J?.4 (Pin_4)
- net SCL3: now also J?.6 (Pin_6), J?.6 (Pin_6)
- net SDA3: now also J?.5 (Pin_5), J?.5 (Pin_5)
- net VBUS: now also J?.10 (Pin_10), J?.10 (Pin_10)

Commit message: Added proper connectors and added traces
Parts:
- J1: renamed from J?; footprint (none) -> batteryboard:SAMTEC_SLM-110-01-G-S
- J2: renamed from J?; footprint (none) -> batteryboard:SAMTEC-FTS-105-01-X-DV
Connections:
- net +3V3: now also J1.03 (Pin_3); no longer J1.3 (Pin_3)
- net BATT_N_SW: now also J1.02 (Pin_2); no longer J1.2 (Pin_2)
- net BATT_P: now also J1.09 (Pin_9); no longer J1.9 (Pin_9)
- net BATT_P_SW: now also J1.01 (Pin_1); no longer J1.1 (Pin_1)
- net COIL_N: now also J1.08 (Pin_8); no longer J1.8 (Pin_8)
- net COIL_P: now also J1.07 (Pin_7); no longer J1.7 (Pin_7)
- net GND: now also J1.04 (Pin_4); no longer J1.4 (Pin_4)
- net SCL3: now also J1.06 (Pin_6); no longer J1.6 (Pin_6)
- net SDA3: now also J1.05 (Pin_5); no longer J1.5 (Pin_5)
Changed lines of the file:
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@@
   (symbol (lib_id "Connector_Generic:Conn_02x05_Odd_Even") (at 165.1 50.8 0) (unit 1)
     (in_bom yes) (on_board yes) (fields_autoplaced)
-    (property "Reference" "J?" (id 0) (at 166.37 39.37 0))
+    (property "Reference" "J2" (id 0) (at 166.37 39.37 0))
     (property "Value" "Conn_02x05_Odd_Even" (id 1) (at 166.37 41.91 0))
-    (property "Footprint" "" (id 2) (at 165.1 50.8 0)
+    (property "Footprint" "batteryboard:SAMTEC-FTS-105-01-X-DV" (id 2) (at 165.1 50.8 0)
       (effects (font (size 1.27 1.27)) hide)
     )
@@
   (symbol (lib_id "Connector_Generic:Conn_01x10") (at 73.66 48.26 0) (mirror y) (unit 1)
     (in_bom yes) (on_board yes) (fields_autoplaced)
-    (property "Reference" "J?" (id 0) (at 73.66 31.75 0))
+    (property "Reference" "J1" (id 0) (at 73.66 31.75 0))
     (property "Value" "Conn_01x10" (id 1) (at 73.66 34.29 0))
-    (property "Footprint" "" (id 2) (at 73.66 48.26 0)
+    (property "Footprint" "batteryboard:SAMTEC_SLM-110-01-G-S" (id 2) (at 71.12 35.56 0)
       (effects (font (size 1.27 1.27)) hide)
     )
@@
       (effects (font (size 1.27 1.27)) hide)
     )
-    (pin "1")
+    (pin "01")
     (pin "10")
-    (pin "2")
-    (pin "3")
-    (pin "4")
-    (pin "5")
-    (pin "6")
-    (pin "7")
-    (pin "8")
-    (pin "9")
+    (pin "02")
+    (pin "03")
+    (pin "04")
+    (pin "05")
+    (pin "06")
+    (pin "07")
+    (pin "08")
+    (pin "09")
   )
   (sheet_instances
@@
       (reference "H4") (unit 1) (value "MountingHole_Pad") (footprint "mainboard:MountingHole")
     )
+    (path "/f04224a8-ae30-44b3-a012-c883be8c361b"
+      (reference "J1") (unit 1) (value "Conn_01x10") (footprint "batteryboard:SAMTEC_SLM-110-01-G-S")
+    )
     (path "/cc451705-64aa-4852-a9e4-e56ff8e107b4"
-      (reference "J?") (unit 1) (value "Conn_02x05_Odd_Even") (footprint "")
-    )
-    (path "/f04224a8-ae30-44b3-a012-c883be8c361b"
-      (reference "J?") (unit 1) (value "Conn_01x10") (footprint "")
+      (reference "J2") (unit 1) (value "Conn_02x05_Odd_Even") (footprint "batteryboard:SAMTEC-FTS-105-01-X-DV")
     )
   )

Commit message: Fixes and cleanup
Parts:
- J1: footprint batteryboard:SAMTEC_SLM-110-01-G-S -> batteryboard:SAMTEC_TMS-110-01-G-S
- J2: footprint batteryboard:SAMTEC-FTS-105-01-X-DV -> batteryboard:FTS-105-XX-YY-DV-A
Connections:
- net +3V3: now also J1.04 (Pin_4); no longer J1.03 (Pin_3)
- net BATT_P: now also J1.01 (Pin_1); no longer J1.09 (Pin_9)
- net BATT_P_SW: now also J1.03 (Pin_3); no longer J1.01 (Pin_1)
- net GND: now also J1.07 (Pin_7); no longer J1.04 (Pin_4)
- net SCL3: now also J1.05 (Pin_5); no longer J1.06 (Pin_6)
- net SDA3: now also J1.06 (Pin_6); no longer J1.05 (Pin_5)
- net COIL_N renamed COIL5_N
- net COIL5_N: now also J1.10 (Pin_10); no longer J1.08 (Pin_8)
- net COIL_P renamed COIL5_P
- net COIL5_P: now also J1.09 (Pin_9); no longer J1.07 (Pin_7)
- net VBUS renamed VUSB
- net VUSB: now also J1.08 (Pin_8); no longer J1.10 (Pin_10)
Other:
- moved on the sheet: H1, H2, H3, H4, J1, J2

Commit message: Recheck boards and re-export models
Parts:
- J1: value Conn_01x10 -> SLM-110-01-G-S
- J2: value Conn_02x05_Odd_Even -> FTS-105-01-L-DV-A
Connections:
- net +3V3: now also J1.4 (Pin_4); no longer J1.04 (Pin_4)
- net BATT_N_SW: now also J1.2 (Pin_2); no longer J1.02 (Pin_2)
- net BATT_P: now also J1.1 (Pin_1); no longer J1.01 (Pin_1)
- net BATT_P_SW: now also J1.3 (Pin_3); no longer J1.03 (Pin_3)
- net COIL5_P: now also J1.9 (Pin_9); no longer J1.09 (Pin_9)
- net GND: now also J1.7 (Pin_7); no longer J1.07 (Pin_7)
- net SCL3: now also J1.5 (Pin_5); no longer J1.05 (Pin_5)
- net SDA3: now also J1.6 (Pin_6); no longer J1.06 (Pin_6)
- net VUSB: now also J1.8 (Pin_8); no longer J1.08 (Pin_8)
Changed lines of the file:
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@@
   (symbol (lib_id "Mechanical:MountingHole_Pad") (at 95.631 93.98 90) (unit 1)
     (in_bom yes) (on_board yes)
-    (property "Reference" "H1" (id 0) (at 83.439 91.948 90))
-    (property "Value" "MountingHole_Pad" (id 1) (at 83.439 94.4849 90))
+    (property "Reference" "H1" (id 0) (at 90.678 92.964 90))
+    (property "Value" "MountingHole_Pad" (id 1) (at 83.312 95.123 90))
     (property "Footprint" "mainboard:MountingHole" (id 2) (at 95.631 93.98 0)
       (effects (font (size 1.27 1.27)) hide)
@@
   (symbol (lib_id "Mechanical:MountingHole_Pad") (at 113.284 88.646 90) (unit 1)
     (in_bom yes) (on_board yes)
-    (property "Reference" "H3" (id 0) (at 132.207 86.614 90))
-    (property "Value" "MountingHole_Pad" (id 1) (at 132.207 89.1509 90))
+    (property "Reference" "H3" (id 0) (at 124.841 87.376 90))
+    (property "Value" "MountingHole_Pad" (id 1) (at 132.207 89.535 90))
     (property "Footprint" "mainboard:MountingHole" (id 2) (at 113.284 88.646 0)
       (effects (font (size 1.27 1.27)) hide)
@@
   (symbol (lib_id "Mechanical:MountingHole_Pad") (at 113.284 94.107 90) (unit 1)
     (in_bom yes) (on_board yes)
-    (property "Reference" "H4" (id 0) (at 132.207 92.075 90))
-    (property "Value" "MountingHole_Pad" (id 1) (at 132.207 94.6119 90))
+    (property "Reference" "H4" (id 0) (at 124.968 93.218 90))
+    (property "Value" "MountingHole_Pad" (id 1) (at 132.334 95.25 90))
     (property "Footprint" "mainboard:MountingHole" (id 2) (at 113.284 94.107 0)
       (effects (font (size 1.27 1.27)) hide)
@@
   (symbol (lib_id "Mechanical:MountingHole_Pad") (at 95.758 88.646 90) (unit 1)
     (in_bom yes) (on_board yes)
-    (property "Reference" "H2" (id 0) (at 83.566 86.6171 90))
-    (property "Value" "MountingHole_Pad" (id 1) (at 83.566 89.154 90))
+    (property "Reference" "H2" (id 0) (at 90.805 87.249 90))
+    (property "Value" "MountingHole_Pad" (id 1) (at 83.439 89.408 90))
     (property "Footprint" "mainboard:MountingHole" (id 2) (at 95.758 88.646 0)
       (effects (font (size 1.27 1.27)) hide)
@@
   )
   (symbol (lib_id "Connector_Generic:Conn_02x05_Odd_Even") (at 150.368 63.373 0) (unit 1)
-    (in_bom yes) (on_board yes) (fields_autoplaced)
-    (property "Reference" "J2" (id 0) (at 151.638 51.943 0))
-    (property "Value" "Conn_02x05_Odd_Even" (id 1) (at 151.638 54.483 0))
+    (in_bom yes) (on_board yes)
+    (property "Reference" "J2" (id 0) (at 151.638 55.499 0))
+    (property "Value" "FTS-105-01-L-DV-A" (id 1) (at 151.638 71.501 0))
     (property "Footprint" "batteryboard:FTS-105-XX-YY-DV-A" (id 2) (at 150.368 63.373 0)
       (effects (font (size 1.27 1.27)) hide)
@@
   )
   (symbol (lib_id "Connector_Generic:Conn_01x10") (at 51.943 61.341 0) (mirror y) (unit 1)
-    (in_bom yes) (on_board yes) (fields_autoplaced)
-    (property "Reference" "J1" (id 0) (at 51.943 44.831 0))
-    (property "Value" "Conn_01x10" (id 1) (at 51.943 47.371 0))
+    (in_bom yes) (on_board yes)
+    (property "Reference" "J1" (id 0) (at 51.943 48.387 0))
+    (property "Value" "SLM-110-01-G-S" (id 1) (at 51.943 77.089 0))
     (property "Footprint" "batteryboard:SAMTEC_TMS-110-01-G-S" (id 2) (at 49.403 48.641 0)
       (effects (font (size 1.27 1.27)) hide)
@@
       (effects (font (size 1.27 1.27)) hide)
     )
-    (pin "01")
-    (pin "02")
-    (pin "03")
-    (pin "04")
-    (pin "05")
-    (pin "06")
-    (pin "07")
-    (pin "08")
-    (pin "09")
+    (pin "1")
     (pin "10")
+    (pin "2")
+    (pin "3")
+    (pin "4")
+    (pin "5")
+    (pin "6")
+    (pin "7")
+    (pin "8")
+    (pin "9")
   )
   (sheet_instances
@@
     )
     (path "/f04224a8-ae30-44b3-a012-c883be8c361b"
-      (reference "J1") (unit 1) (value "Conn_01x10") (footprint "batteryboard:SAMTEC_TMS-110-01-G-S")
+      (reference "J1") (unit 1) (value "SLM-110-01-G-S") (footprint "batteryboard:SAMTEC_TMS-110-01-G-S")
     )
     (path "/cc451705-64aa-4852-a9e4-e56ff8e107b4"
-      (reference "J2") (unit 1) (value "Conn_02x05_Odd_Even") (footprint "batteryboard:FTS-105-XX-YY-DV-A")
+      (reference "J2") (unit 1) (value "FTS-105-01-L-DV-A") (footprint "batteryboard:FTS-105-XX-YY-DV-A")
     )
   )
