File: batteryboard-bottom/batteryboard-bottom.kicad_pcb (KiCad board)
At the start: 2 copper layers, 46.8 x 46.8 mm, 7 parts, among them J1 SLM-110-01-G-S, J2 FTS-105-01-L-DV-A

Commit message: Some changes
Parts:
- J1: value SLM-110-01-G-S -> SFC-110-T2-F-D-A; footprint batteryboard:SAMTEC_TMS-110-01-G-S -> mainboard:SAMTEC_SFC-110-T2-F-D-A-TR
- J2: value FTS-105-01-L-DV-A -> FTS-107-01-L-DV-A; footprint batteryboard:FTS-105-XX-YY-DV-A -> batteryboard:SAMTEC-FTS-107-01-X-DV-A
- moved J1 2.70 mm to (133.5, 105.2), turned to -90 degrees
- turned J2 to -90 degrees
Connections:
- J1 pad 1: BATT_P -> COIL6_N
- J1 pad 10: COIL5_N -> +3V3
- J1 pad 2: BATT_N_SW -> COIL5_P
- J1 pad 3: BATT_P_SW -> GND
- J1 pad 4: +3V3 -> GND
- J1 pad 5: SCL3 -> UART_TX
- J1 pad 6: SDA3 -> SCL1
- J1 pad 7: GND -> UART_RX
- J1 pad 8: VUSB -> SDA1
- J1 pad 9: COIL5_P -> +3V3
- J2 pad 1: BATT_P_SW -> GND
- J2 pad 10: VUSB -> BATT_P
- J2 pad 3: +3V3 -> GND
- J2 pad 4: GND -> BATT_N_SW
- J2 pad 5: SDA3 -> +3V3
- J2 pad 6: SCL3 -> BATT_P_SW
- J2 pad 7: COIL5_P -> +3V3
- J2 pad 8: COIL5_N -> BATT_P_SW
- J2 pad 9: BATT_P -> SCL1
Routing:
- net BATT_P: track 40.9 -> 0.00 mm
- net COIL5_P: track 25.2 -> 0.00 mm
- net SCL3: track 23.7 -> 0.00 mm, vias 1 -> 0
- net SCL1: track 0.00 -> 19.0 mm, vias 0 -> 1
- net +3V3: track 18.8 -> 0.00 mm, vias 1 -> 4
- net SDA3: track 16.7 -> 0.00 mm, vias 1 -> 0
- net SDA1: track 0.00 -> 16.4 mm, vias 0 -> 1
- net BATT_P_SW: track 7.51 -> 0.00 mm, vias 3 -> 0
- net COIL5_N: track 11.9 -> 8.40 mm
- net VUSB: track 0.42 -> 0.00 mm, vias 1 -> 0
- net GND: vias 2 -> 1
- added copper zone on B.Cu, net +3V3
- added copper zone on B.Cu, net BATT_N_SW
- added copper zone on B.Cu, net BATT_P
- removed copper zone on F.Cu, net BATT_N_SW
- removed copper zone on B.Cu, net VUSB
Other:
- outline, holes or cut-outs redrawn
- board text added: "Rev B2/01"
- board text removed: "Bottom Battery Board"
- board text removed: "Rev B1/03"

Commit message: B2/01 Updates
Routing:
- net COIL5_P: track 0.00 -> 17.3 mm
- net SCL1: track 19.0 -> 18.2 mm
- net GND: vias 1 -> 3
- net BATT_P_SW: vias 0 -> 4
- net BATT_P: vias 0 -> 4
- net BATT_N_SW: vias 0 -> 4
Other:
- board text added: "09-OCT-22"
- board text removed: "06-SEP-22"

Commit message: Minor updates and exported STEP / BOM
Parts:
- moved J2 2.03 mm to (133.7, 92.1)
Routing:
- net SDA1: track 16.4 -> 12.6 mm, vias 1 -> 3
- net SCL1: track 18.2 -> 15.3 mm, vias 1 -> 3
- net COIL5_N: track 8.09 -> 5.61 mm
- net GND: vias 3 -> 5
Other:
- outline, holes or cut-outs redrawn
- board text added: "06-NOV-22"
- board text removed: "09-OCT-22"
