File: batteryboard-bottom/Bus Protection.kicad_sch (KiCad schematic)
At the start: 18 parts, among them Q1 NX3008NBKS, Q2 MBT2222ADW1T1, Q3 NX3008NBKS, Q4 MBT2222ADW1T1

Commit message: Rev B3/02 updates
Other:
- company: (none) -> RExLab Carnegie Mellon University
- title: (none) -> PyCubed Mini
Changed lines of the file:
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@@
 (kicad_sch (version 20230121) (generator eeschema)
   (paper "A4")
+  (title_block
+    (title "PyCubed Mini")
+    (date "2023-04-12")
+    (rev "B3/02")
+    (company "RExLab Carnegie Mellon University")
+    (comment 1 "N. Khera")
+    (comment 2 "Z. Manchester")
+  )
   (junction (at 80.264 117.856) (diameter 0) (color 0 0 0 0)
   )

Commit message: Rev B3/03 updates
Parts:
- added C8, C9: 10nF, Capacitor_SMD:C_0603_1608Metric, symbol Device:C
- added Q5, Q7: NX3008NBKS, Package_TO_SOT_SMD:SOT-363_SC-70-6, symbol mainboard:NX3008NBKS
- added Q6, Q8: MBT2222ADW1T1, Package_TO_SOT_SMD:SOT-363_SC-70-6, symbol Transistor_BJT:MBT2222ADW1T1
- added R14, R21: 680R, Resistor_SMD:R_0603_1608Metric, symbol Device:R_US
- added R15, R22: 100K, Resistor_SMD:R_0603_1608Metric, symbol Device:R_US
- added R18, R19, R23, R24: 10K, Resistor_SMD:R_0603_1608Metric, symbol Device:R_US
- added R20, R25: 200K, Resistor_SMD:R_0603_1608Metric, symbol Device:R_US
- added R26, R27: DNI (0R), Resistor_SMD:R_0603_1608Metric, symbol Device:R_US
Connections:
- net +3V3: now also R15.1, R18.1, R19.1, R22.1, R23.1, R24.1
- net GND: now also C8.2, C9.2, Q5.1 (S2), Q5.4 (S1), Q7.1 (S2), Q7.4 (S1)
- net SCL1: now also Q6.1 (E1), Q6.3 (C2), R26.2
- net SDA1: now also Q8.1 (E1), Q8.3 (C2), R27.2
- new net: C9.1, Q7.5 (G1), R25.2
- new net: Q5.2 (G2), Q5.3 (D2), R15.2
- new net: C8.1, Q5.5 (G1), R20.2
- new net: Q7.2 (G2), Q7.3 (D2), R22.2
- new net: Q7.6 (D1), Q8.5 (B2), R21.2, R23.2
- new net: Q8.2 (B1), R21.1
- new net: Q5.6 (D1), Q6.5 (B2), R14.2, R18.2
- new net: Q6.2 (B1), R14.1
- new net SCL_IMU: Q6.4 (E2), Q6.6 (C1), R19.2, R20.1, R26.1
- new net SDA_IMU: Q8.4 (E2), Q8.6 (C1), R24.2, R25.1, R27.1
Other:
- note added: "Current Sensor Jumpers"
- note added: "I2C Bus Protection - IMU"
- note added: "IMU Jumpers"
- note removed: "Light Sensor Jumpers"
- moved on the sheet: C12, C13, Q1A, Q1B, Q2A, Q2B, Q3A, Q3B, Q4A, Q4B, R19, R20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
