File: batteryboard-middle/batteryboard-middle.kicad_pcb (KiCad board)
At the start: 2 copper layers, 46.8 x 46.8 mm, 10 parts, among them J1 Conn_01x02, J2 Conn_01x02, J4 FLE-110-01-G-DV-A, J5 FTS-110-01-L-DV-A, J6 FTS-110-01-L-DV-A

Commit message: Fixed Broken Merge
Parts:
- removed J5: FTS-110-01-L-DV-A, batteryboard:Battery Pads
- removed J6: FTS-110-01-L-DV-A, batteryboard:SAMTEC-FTS-110-01-X-DV-A
- added J3: Conn_01x02, batteryboard:Battery Pads, F.Cu at (146.8, 121.1)
- J1: value Conn_01x02 -> FLE-105-01-G-DV-A; footprint batteryboard:Battery Pads -> batteryboard:SAMTEC_FLE-105-01-G-DV-A; moved to B.Cu
- J4: value FLE-110-01-G-DV-A -> FTS-105-01-L-DV-A; footprint mainboard:SAMTEC_FLE-110-01-G-DV-A -> batteryboard:FTS-105-XX-YY-DV-A; moved to F.Cu
- moved H3 43.2 mm to (126.9, 120.5), turned to -90 degrees
- moved H4 43.2 mm to (126.9, 80.7), turned to -90 degrees
- moved J1 39.1 mm to (127.8, 89.0), turned to 90 degrees
- moved H1 36.4 mm to (166.7, 80.7), turned to -90 degrees
- moved H2 36.4 mm to (166.7, 120.5), turned to -90 degrees
- moved J4 13.6 mm to (127.8, 89.0), turned to 90 degrees
Connections:
- J4 pad 1: BATT_P -> unconnected-(J4-Pad1)
- J4 pad 10: MOSI -> VBUS
- J4 pad 2: BATT_P_SW -> unconnected-(J4-Pad2)
- J4 pad 3: unconnected-(J4-Pad3) -> +3V3
- J4 pad 4: BATT_N_SW -> GND
- J4 pad 5: SD_CS -> SDA3
- J4 pad 6: CAM_EN -> SCL3
- J4 pad 7: SCK -> COIL_P
- J4 pad 8: MISO -> COIL_N
- J4 pad 9: CAM_CS -> BATT_P
Routing:
- net unconnected-(J3-Pad5): vias 1 -> 0
- net unconnected-(J3-Pad3): vias 1 -> 0
- net unconnected-(J3-Pad1): vias 1 -> 0
- net VUSB: vias 1 -> 0
- net VBUS: vias 0 -> 1
- net SDA3: vias 0 -> 1
- net SCL3: vias 0 -> 1
- net COIL_P: vias 0 -> 1
- net COIL_N: vias 0 -> 1
- net BURN1: vias 1 -> 0

Commit message: Some changes
Parts:
- J1: value FLE-105-01-G-DV-A -> FLE-107-01-G-DV-A; footprint batteryboard:SAMTEC_FLE-105-01-G-DV-A -> batteryboard:SAMTEC_FLE-107-01-G-DV-A
- J4: value FTS-105-01-L-DV-A -> FTS-107-01-L-DV-A; footprint batteryboard:FTS-105-XX-YY-DV-A -> batteryboard:SAMTEC-FTS-107-01-X-DV-A
- turned J1 to -90 degrees
- turned J4 to -90 degrees
Connections:
- J1 pad 1: BATT_P_SW -> GND
- J1 pad 10: VBUS -> BATT_N_SW
- J1 pad 2: BATT_N_SW -> GND
- J1 pad 4: GND -> BATT_P_SW
- J1 pad 5: SDA3 -> +3V3
- J1 pad 6: SCL3 -> BATT_P_SW
- J1 pad 7: COIL_P -> BATT_P
- J1 pad 8: COIL_N -> BATT_N_SW
- J4 pad 1: unconnected-(J4-Pad1) -> GND
- J4 pad 10: VBUS -> BATT_N_SW
- J4 pad 2: unconnected-(J4-Pad2) -> GND
- J4 pad 4: GND -> BATT_P_SW
- J4 pad 5: SDA3 -> +3V3
- J4 pad 6: SCL3 -> BATT_P_SW
- J4 pad 7: COIL_P -> BATT_P
- J4 pad 8: COIL_N -> BATT_N_SW
Routing:
- net BATT_P: track 16.2 -> 0.00 mm, vias 3 -> 2
- net BATT_P_SW: track 10.3 -> 0.00 mm, vias 8 -> 7
- net BATT_N_SW: track 9.80 -> 0.00 mm, vias 5 -> 7
- net VBUS: vias 1 -> 0
- net SDA3: vias 1 -> 0
- net SDA1: vias 0 -> 1
- net SCL3: vias 1 -> 0
- net SCL1: vias 0 -> 1
- net COIL_P: vias 1 -> 0
- net COIL_N: vias 1 -> 0
- net COIL5_P: vias 0 -> 1
- net COIL5_N: vias 0 -> 1
- net +3V3: vias 1 -> 2
- added copper zone on B.Cu, net +3V3
- added copper zone on F.Cu, net +3V3
- added copper zone on F.Cu, net BATT_N_SW
- added copper zone on B.Cu, net BATT_P
- added copper zone on F.Cu, net BATT_P
- added copper zone on B.Cu, net BATT_P_SW
Other:
- board text added: "Rev B2/01"
- board text removed: "Middle Battery Board"
- board text removed: "Rev B1/03"

Commit message: B2/01 Updates
Connections:
- J1 pad 10: BATT_N_SW -> BATT_P
- J1 pad 11: SCL1 -> SDA1
- J1 pad 12: COIL5_P -> BATT_P
- J1 pad 13: SDA1 -> COIL5_P
- J1 pad 2: GND -> BATT_N_SW
- J1 pad 3: +3V3 -> GND
- J1 pad 4: BATT_P_SW -> BATT_N_SW
- J1 pad 7: BATT_P -> +3V3
- J1 pad 8: BATT_N_SW -> BATT_P_SW
- J1 pad 9: BATT_P -> SCL1
- J4 pad 10: BATT_N_SW -> BATT_P
- J4 pad 11: SCL1 -> SDA1
- J4 pad 12: COIL5_P -> BATT_P
- J4 pad 13: SDA1 -> COIL5_P
- J4 pad 2: GND -> BATT_N_SW
- J4 pad 3: +3V3 -> GND
- J4 pad 4: BATT_P_SW -> BATT_N_SW
- J4 pad 7: BATT_P -> +3V3
- J4 pad 8: BATT_N_SW -> BATT_P_SW
- J4 pad 9: BATT_P -> SCL1
Other:
- board text added: "09-OCT-22"
- board text removed: "06-SEP-22"

Commit message: Minor Schematic Updates
Routing:
- net BATT_P_SW: vias 7 -> 9
- net BATT_P: vias 2 -> 4
- net BATT_N_SW: vias 7 -> 9
Changed lines of the file:
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@@
     (effects (font (size 0.635 0.635) (thickness 0.1524)) (justify right))
   )
-  (via (at 129.62 88.98) (size 0.762) (drill 0.381) (layers "F.Cu" "B.Cu") (net 1))
+  (via (at 130.07 88.98) (size 0.762) (drill 0.381) (layers "F.Cu" "B.Cu") (net 1))
   (via (at 150.9 121.8) (size 0.8) (drill 0.4) (layers "F.Cu" "B.Cu") (net 1))
   (via (at 148.7062 120.3926) (size 0.8) (drill 0.4) (layers "F.Cu" "B.Cu") (net 1))
@@
   (via (at 150.9 120.4) (size 0.8) (drill 0.4) (layers "F.Cu" "B.Cu") (net 1))
   (via (at 149.8 121.1) (size 0.8) (drill 0.4) (layers "F.Cu" "B.Cu") (net 1))
-  (via (at 129.62 87.71) (size 0.762) (drill 0.381) (layers "F.Cu" "B.Cu") (net 1))
+  (via (at 129.17 87.72) (size 0.762) (drill 0.381) (layers "F.Cu" "B.Cu") (net 1))
+  (via (at 129.17 88.99) (size 0.762) (drill 0.381) (layers "F.Cu" "B.Cu") (net 1))
+  (via (at 130.07 87.71) (size 0.762) (drill 0.381) (layers "F.Cu" "B.Cu") (net 1))
   (via (at 145 121.8) (size 0.8) (drill 0.4) (layers "F.Cu" "B.Cu") (net 2))
   (via (at 142.6 120.4) (size 0.8) (drill 0.4) (layers "F.Cu" "B.Cu") (net 2))
   (via (at 145 120.4) (size 0.8) (drill 0.4) (layers "F.Cu" "B.Cu") (net 2))
-  (via (at 129.62 86.44) (size 0.762) (drill 0.381) (layers "F.Cu" "B.Cu") (net 2))
-  (via (at 129.6 85.17) (size 0.762) (drill 0.381) (layers "F.Cu" "B.Cu") (net 2))
+  (via (at 129.15 85.18) (size 0.762) (drill 0.381) (layers "F.Cu" "B.Cu") (net 2))
+  (via (at 129.17 86.45) (size 0.762) (drill 0.381) (layers "F.Cu" "B.Cu") (net 2))
+  (via (at 130.07 86.44) (size 0.762) (drill 0.381) (layers "F.Cu" "B.Cu") (net 2))
+  (via (at 130.05 85.17) (size 0.762) (drill 0.381) (layers "F.Cu" "B.Cu") (net 2))
   (via (at 143.8 121.1) (size 0.8) (drill 0.4) (layers "F.Cu" "B.Cu") (net 2))
   (via (at 142.6 121.8) (size 0.8) (drill 0.4) (layers "F.Cu" "B.Cu") (net 2))
@@
   (via (at 125.94 88.98) (size 0.762) (drill 0.381) (layers "F.Cu" "B.Cu") (net 4))
   (via (at 125.94 87.71) (size 0.762) (drill 0.381) (layers "F.Cu" "B.Cu") (net 4))
-  (via (at 129.62 90.25) (size 0.762) (drill 0.381) (layers "F.Cu" "B.Cu") (net 5))
-  (via (at 129.62 91.52) (size 0.762) (drill 0.381) (layers "F.Cu" "B.Cu") (net 5))
+  (via (at 129.17 91.53) (size 0.762) (drill 0.381) (layers "F.Cu" "B.Cu") (net 5))
+  (via (at 129.17 90.26) (size 0.762) (drill 0.381) (layers "F.Cu" "B.Cu") (net 5))
+  (via (at 130.07 90.25) (size 0.762) (drill 0.381) (layers "F.Cu" "B.Cu") (net 5))
+  (via (at 130.07 91.52) (size 0.762) (drill 0.381) (layers "F.Cu" "B.Cu") (net 5))
   (via (at 125.95 91.52) (size 0.762) (drill 0.381) (layers "F.Cu" "B.Cu") (net 6))
   (via (at 125.94 90.25) (size 0.762) (drill 0.381) (layers "F.Cu" "B.Cu") (net 7))

Commit message: Minor updates and exported STEP / BOM
Parts:
- moved J1 2.03 mm to (127.8, 91.0)
- moved J4 2.03 mm to (127.8, 91.0)
Other:
- outline, holes or cut-outs redrawn
- board text added: "06-NOV-22"
- board text removed: "09-OCT-22"
