File: batteryboard-top/batteryboard-top.kicad_pcb (KiCad board)
At the start: 2 copper layers, 46.8 x 46.8 mm, 7 parts, among them J1 FLE-105-01-G-DV-A, J2 FLE-105-01-G-DV-A

Commit message: Exported Files
Other:
- board text added: "Aleksei Seletskiy Gaurav Savant Jacob Willis Karissa Barbu Krrish Jain Max Holliday Neil Khera Paulo Fisch Yashika Batra Zac Manchester"
- board text removed: "Aleksei Seletskiy Gaurav Savant Jacob Willis Krrish Jain Neil Khera Paulo Fisch Yashika Batra Zac Manchester"
Changed lines of the file:
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@@
       (psnegative false)
       (psa4output false)
-      (plotreference true)
+      (plotreference false)
       (plotvalue true)
       (plotinvisibletext false)
@@
       (drillshape 0)
       (scaleselection 1)
-      (outputdirectory "../gerbers/batteryboard-top (07-06-22)/")
+      (outputdirectory "../gerbers/batteryboard-top (09-09-22)/")
     )
   )
@@
     (effects (font (size 1 1) (thickness 0.15) italic) (justify mirror))
   )
-  (gr_text "Aleksei Seletskiy\nGaurav Savant\nJacob Willis\nKrrish Jain\nNeil Khera\nPaulo Fisch\nYashika Batra\nZac Manchester" (at 150.4 92.7) (layer "F.SilkS")
+  (gr_text "Aleksei Seletskiy\nGaurav Savant\nJacob Willis\nKarissa Barbu\nKrrish Jain\nMax Holliday\nNeil Khera\nPaulo Fisch\nYashika Batra\nZac Manchester" (at 150.4 92.7) (layer "F.SilkS")
     (effects (font (size 0.762 0.762) (thickness 0.127)))
   )
@@
       47eb5539-25ae-4f84-af49-4174bb1ebee0
       48d6239e-e098-424b-bc8f-3355174d069c
-      4b7db72b-f164-47a4-a269-3726f03ee677
       4daca37e-fbee-4ad6-91ce-78585073fe34
       4ee1d11d-cc0c-4a88-a80e-1cc592c33ff5
@@
       9978a360-cbd0-44a2-b0c5-5128e5cb2abd
       9fe0348e-1c03-494b-b65b-99dc55261104
-      a05dbeca-7a55-48d7-9d1e-2fb90b14ecdd
       a3a4b9ea-8328-4cd5-b06b-56fa0cf4fee6
       aa307439-b9d3-4aa9-93dc-e2d437f14fe6
@@
       bc3fbea7-9841-483b-b043-08b9d50af1b5
       cc22c5f4-6a68-4464-9585-ac59c4269649
-      d506b9e0-5dbd-4ee9-b406-2356292be30f
       e94a2169-66e2-48f7-9e02-eaebd9f3b88f
       ea73d19a-4016-4e47-b917-817c1581977b
       ecf6b1f2-75e6-4299-8bae-cd90b584dffe
       f44265a9-dd2e-417b-b3c5-99c145d344f5
-      fce9f559-6c56-4f15-b0b6-32a3d29676cd
       fe0898d7-33bf-41fa-9ede-79bb4e91d959
     )

Commit message: Some changes
Parts:
- J1: value FLE-105-01-G-DV-A -> FLE-107-01-G-DV-A; footprint batteryboard:SAMTEC_FLE-105-01-G-DV-A -> batteryboard:SAMTEC_FLE-107-01-G-DV-A
- turned J1 to -90 degrees
- turned J2 to -90 degrees
Connections:
- J1 pad 1: unconnected-(J1-Pad1) -> GND
- J1 pad 10: VBUS -> unconnected-(J1-Pad10)
- J1 pad 2: unconnected-(J1-Pad2) -> GND
- J1 pad 4: GND -> unconnected-(J1-Pad4)
- J1 pad 5: SDA3 -> +3V3
- J1 pad 6: SCL3 -> unconnected-(J1-Pad6)
- J1 pad 7: COIL_P -> BATT_P
- J1 pad 8: COIL_N -> unconnected-(J1-Pad8)
- J2 pad 1: unconnected-(J2-Pad1) -> GND
- J2 pad 10: VBUS -> SDA1
- J2 pad 2: unconnected-(J2-Pad2) -> +3V3
- J2 pad 3: +3V3 -> GND
- J2 pad 4: GND -> BATT_P
- J2 pad 5: SDA3 -> unconnected-(J2-Pad5)
- J2 pad 6: SCL3 -> BATT_P
- J2 pad 7: COIL_P -> COIL5_P
- J2 pad 8: COIL_N -> SCL1
- J2 pad 9: BATT_P -> COIL5_N
Routing:
- net SCL3: track 46.1 -> 0.00 mm, vias 1 -> 0
- net COIL_N: track 45.4 -> 0.00 mm, vias 1 -> 0
- net VBUS: track 35.5 -> 0.00 mm, vias 1 -> 0
- net BATT_P: track 34.7 -> 0.00 mm
- net COIL5_P: track 0.00 -> 29.7 mm, vias 0 -> 1
- net COIL5_N: track 0.00 -> 29.7 mm, vias 0 -> 1
- net SCL1: track 0.00 -> 29.4 mm, vias 0 -> 1
- net SDA1: track 0.00 -> 29.3 mm, vias 0 -> 1
- net SDA3: track 26.1 -> 0.00 mm, vias 1 -> 0
- net +3V3: track 26.1 -> 0.00 mm, vias 1 -> 3
- net COIL_P: track 26.1 -> 0.00 mm, vias 1 -> 0
- net GND: vias 3 -> 4
- added copper zone on B.Cu, net +3V3
- added copper zone on F.Cu, net +3V3
- added copper zone on B.Cu, net BATT_P
- added copper zone on F.Cu, net BATT_P
Other:
- board text added: "Aleksei Seletskiy Gaurav Savant Jacob Willis Jeffery John Karissa Barbu Krrish Jain Max Holliday Neil Khera Paulo Fisch Yashika Batra Zac Manchester"
- board text added: "Rev B2/01"
- board text removed: "Aleksei Seletskiy Gaurav Savant Jacob Willis Karissa Barbu Krrish Jain Max Holliday Neil Khera Paulo Fisch Yashika Batra Zac Manchester"
- board text removed: "Rev B1/03"
- board text removed: "Top Battery Board"

Commit message: B2/01 Updates
Connections:
- J1 pad 10: unconnected-(J1-Pad10) -> BATT_P
- J1 pad 11: SCL1 -> SDA1
- J1 pad 12: COIL5_P -> BATT_P
- J1 pad 13: SDA1 -> COIL5_P
- J1 pad 2: GND -> unconnected-(J1-Pad2)
- J1 pad 3: +3V3 -> GND
- J1 pad 7: BATT_P -> +3V3
- J1 pad 9: BATT_P -> SCL1
- J2 pad 7: COIL5_P -> COIL5_N
- J2 pad 9: COIL5_N -> COIL5_P
Routing:
- net COIL5_P: track 29.7 -> 36.9 mm
- net COIL5_N: track 29.7 -> 32.7 mm
- net SDA1: track 29.3 -> 30.4 mm
- net SCL1: track 29.4 -> 30.2 mm
- net BATT_P: vias 3 -> 4
Other:
- board text added: "09-OCT-22"
- board text removed: "06-SEP-22"

Commit message: Minor updates and exported STEP / BOM
Parts:
- moved J1 2.03 mm to (131.4, 86.9)
Routing:
- net SDA1: track 30.4 -> 29.3 mm
- net SCL1: track 30.2 -> 29.3 mm
- net COIL5_P: track 36.9 -> 37.7 mm
- net COIL5_N: track 32.7 -> 33.5 mm
Other:
- outline, holes or cut-outs redrawn
- board text added: "06-NOV-22"
- board text removed: "09-OCT-22"
